File: Eagle/Rover Motor Controller R1/Rover Motor Controller R1.sch (EAGLE design)
At the start: 14 parts, among them U1 ATTINY2313A

Commit message: New Motor Controller Revision
Parts:
- removed SJ1, SJ2, SJ3, SJ4: JUMPER-PAD-2-NOYES_SILK, SparkFun-Passives:JUMPER-PAD-2-NOYES_SILK
- added TP3, TP4, TP5, TP6: TEST-POINT3X4, SparkFun-Passives:TEST-POINT3X4
Connections:
- removed net PD4: SJ1.1, U1.PD4
- removed net PD5: SJ2.1, U1.PD5
- new net PD2: TP3.1, U1.PD2/INT0
- new net PD3: TP4.1, U1.PD3/INT1
- net GND: no longer SJ1.2, SJ2.2, SJ3.2, SJ4.2
- net PB0: now also TP5.1; no longer SJ3.1
- net PB1: now also TP6.1; no longer SJ4.1
- net QEA: now also U1.PD4; no longer U1.PD2/INT0
- net QEB: now also U1.PD5; no longer U1.PD3/INT1
Changed lines of the file:
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@@
 <part name="TP1" library="SparkFun-Passives" deviceset="TEST-POINT" device="3X4"/>
 <part name="TP2" library="SparkFun-Passives" deviceset="TEST-POINT" device="3X4"/>
+<part name="TP3" library="SparkFun-Passives" deviceset="TEST-POINT" device="3X4"/>
+<part name="TP4" library="SparkFun-Passives" deviceset="TEST-POINT" device="3X4"/>
 <part name="GND4" library="supply1" deviceset="GND" device=""/>
+<part name="TP5" library="SparkFun-Passives" deviceset="TEST-POINT" device="3X4"/>
+<part name="TP6" library="SparkFun-Passives" deviceset="TEST-POINT" device="3X4"/>
 <part name="U$1" library="SparkFun-PowerIC" deviceset="V_REG_MIC2920" device=""/>
-<part name="SJ1" library="SparkFun-Passives" deviceset="JUMPER-PAD-2-NO" device="YES_SILK"/>
-<part name="SJ2" library="SparkFun-Passives" deviceset="JUMPER-PAD-2-NO" device="YES_SILK"/>
-<part name="SJ3" library="SparkFun-Passives" deviceset="JUMPER-PAD-2-NO" device="YES_SILK"/>
-<part name="SJ4" library="SparkFun-Passives" deviceset="JUMPER-PAD-2-NO" device="YES_SILK"/>
-<part name="GND5" library="supply1" deviceset="GND" device=""/>
 </parts>
 <sheets>
@@
 <instance part="TP1" gate="G$1" x="134.62" y="68.58"/>
 <instance part="TP2" gate="G$1" x="134.62" y="60.96"/>
+<instance part="TP3" gate="G$1" x="134.62" y="53.34"/>
+<instance part="TP4" gate="G$1" x="134.62" y="45.72"/>
 <instance part="GND4" gate="1" x="73.66" y="63.5"/>
+<instance part="TP5" gate="G$1" x="134.62" y="38.1"/>
+<instance part="TP6" gate="G$1" x="134.62" y="30.48"/>
 <instance part="U$1" gate="G$1" x="73.66" y="73.66"/>
-<instance part="SJ1" gate="G$1" x="139.7" y="53.34"/>
-<instance part="SJ2" gate="G$1" x="139.7" y="45.72"/>
-<instance part="SJ3" gate="G$1" x="139.7" y="38.1"/>
-<instance part="SJ4" gate="G$1" x="139.7" y="30.48"/>
-<instance part="GND5" gate="1" x="147.32" y="20.32"/>
 </instances>
 <busses>
@@
 <pinref part="GND4" gate="1" pin="GND"/>
 </segment>
-<segment>
-<pinref part="SJ1" gate="G$1" pin="2"/>
-<pinref part="GND5" gate="1" pin="GND"/>
-<wire x1="144.78" y1="53.34" x2="147.32" y2="53.34" width="0.1524" layer="91"/>
-<wire x1="147.32" y1="53.34" x2="147.32" y2="45.72" width="0.1524" layer="91"/>
-<pinref part="SJ2" gate="G$1" pin="2"/>
-<wire x1="147.32" y1="45.72" x2="147.32" y2="38.1" width="0.1524" layer="91"/>
-<wire x1="147.32" y1="38.1" x2="147.32" y2="30.48" width="0.1524" layer="91"/>
-<wire x1="147.32" y1="30.48" x2="147.32" y2="22.86" width="0.1524" layer="91"/>
-<wire x1="144.78" y1="45.72" x2="147.32" y2="45.72" width="0.1524" layer="91"/>
-<pinref part="SJ3" gate="G$1" pin="2"/>
-<wire x1="144.78" y1="38.1" x2="147.32" y2="38.1" width="0.1524" layer="91"/>
-<pinref part="SJ4" gate="G$1" pin="2"/>
-<wire x1="144.78" y1="30.48" x2="147.32" y2="30.48" width="0.1524" layer="91"/>
-<junction x="147.32" y="30.48"/>
-<junction x="147.32" y="38.1"/>
-<junction x="147.32" y="45.72"/>
-</segment>
 </net>
 <net name="IN1" class="0">
@@
 </segment>
 <segment>
-<pinref part="U1" gate="G$1" pin="PD2/INT0"/>
-<wire x1="60.96" y1="43.18" x2="58.42" y2="43.18" width="0.1524" layer="91"/>
-<label x="58.42" y="43.18" size="1.778" layer="95" rot="R180"/>
+<pinref part="U1" gate="G$1" pin="PD4"/>
+<wire x1="60.96" y1="38.1" x2="58.42" y2="38.1" width="0.1524" layer="91"/>
+<label x="58.42" y="38.1" size="1.778" layer="95" rot="R180"/>
 </segment>
 </net>
@@
 </segment>
 <segment>
-<pinref part="U1" gate="G$1" pin="PD3/INT1"/>
-<wire x1="60.96" y1="40.64" x2="58.42" y2="40.64" width="0.1524" layer="91"/>
-<label x="58.42" y="40.64" size="1.778" layer="95" rot="R180"/>
+<pinref part="U1" gate="G$1" pin="PD5"/>
+<wire x1="60.96" y1="35.56" x2="58.42" y2="35.56" width="0.1524" layer="91"/>
+<label x="58.42" y="35.56" size="1.778" layer="95" rot="R180"/>
 </segment>
 </net>
@@
 <wire x1="134.62" y1="30.48" x2="132.08" y2="30.48" width="0.1524" layer="91"/>
 <label x="132.08" y="30.48" size="1.778" layer="95" rot="R180"/>
-<pinref part="SJ4" gate="G$1" pin="1"/>
+<pinref part="TP6" gate="G$1" pin="1"/>
 </segment>
 </net>
@@
 <wire x1="134.62" y1="38.1" x2="132.08" y2="38.1" width="0.1524" layer="91"/>
 <label x="132.08" y="38.1" size="1.778" layer="95" rot="R180"/>
-<pinref part="SJ3" gate="G$1" pin="1"/>
+<pinref part="TP5" gate="G$1" pin="1"/>
 </segment>
 </net>
@@
 </segment>
 </net>
-<net name="PD4" class="0">
-<segment>
-<pinref part="U1" gate="G$1" pin="PD4"/>
-<wire x1="60.96" y1="38.1" x2="58.42" y2="38.1" width="0.1524" layer="91"/>
-<label x="58.42" y="38.1" size="1.778" layer="95" rot="R180"/>
+<net name="PD2" class="0">
+<segment>
+<pinref part="U1" gate="G$1" pin="PD2/INT0"/>
+<wire x1="60.96" y1="43.18" x2="58.42" y2="43.18" width="0.1524" layer="91"/>
+<label x="58.42" y="43.18" size="1.778" layer="95" rot="R180"/>
 </segment>
 <segment>
 <wire x1="134.62" y1="53.34" x2="132.08" y2="53.34" width="0.1524" layer="91"/>
 <label x="132.08" y="53.34" size="1.778" layer="95" rot="R180"/>
-<pinref part="SJ1" gate="G$1" pin="1"/>
-</segment>
-</net>
-<net name="PD5" class="0">
-<segment>
-<pinref part="U1" gate="G$1" pin="PD5"/>
-<wire x1="60.96" y1="35.56" x2="58.42" y2="35.56" width="0.1524" layer="91"/>
-<label x="58.42" y="35.56" size="1.778" layer="95" rot="R180"/>
+<pinref part="TP3" gate="G$1" pin="1"/>
+</segment>
+</net>
+<net name="PD3" class="0">
+<segment>
+<pinref part="U1" gate="G$1" pin="PD3/INT1"/>
+<wire x1="60.96" y1="40.64" x2="58.42" y2="40.64" width="0.1524" layer="91"/>
+<label x="58.42" y="40.64" size="1.778" layer="95" rot="R180"/>
 </segment>
 <segment>
 <wire x1="134.62" y1="45.72" x2="132.08" y2="45.72" width="0.1524" layer="91"/>
 <label x="132.08" y="45.72" size="1.778" layer="95" rot="R180"/>
-<pinref part="SJ2" gate="G$1" pin="1"/>
-</segment>
-</net>
+<pinref part="TP4" gate="G$1" pin="1"/>
+</segment>
+</net>
